Commit message: changed robot cloring and added diff drive plugin

File: ros_ws/install/toycar/share/toycar/urdf_description/robot.urdf.xacro (robot description, xacro)
@@ -2,3 +2,4 @@
 <robot xmlns:xacro = "http://ww.ros.org/wiki/xacro" name="robot">
 <xacro:include filename="robot_core0.xacro" />
+<xacro:include filename="diff_drive.xacro" />
 </robot>

File: ros_ws/install/toycar/share/toycar/urdf_description/robot_core.xacro (robot description, xacro)
@@ -41,4 +41,7 @@
         </xacro:inertial_box>
     </link>
+    <gazebo reference = "chassis">
+    <material>Gazebo/White</material>
+    </gazebo>
     <!-- LEFT WHEEL LINK -->
     <joint name="left_wheel_joint" type="continuous">
@@ -64,4 +67,7 @@
         </xacro:inertial_cylinder>
     </link>
+    <gazebo reference = "left_wheel">
+    <material>Gazebo/Grey</material>
+    </gazebo>
     <!-- RIGHT WHEEL LINK -->
     <joint name="right_wheel_joint" type="continuous">
@@ -87,4 +93,7 @@
         </xacro:inertial_cylinder>
     </link>
+    <gazebo reference = "right_wheel">
+    <material>Gazebo/Grey</material>
+    </gazebo>
     <!-- CASTER WHEEL LINK -->
     <joint name="caster_wheel_joint" type="fixed">
@@ -109,3 +118,6 @@
         </xacro:inertial_sphere>
     </link>
+    <gazebo reference = "left_wheel">
+    <material>Gazebo/Grey</material>
+    </gazebo>
 </robot>

File: ros_ws/install/toycar/share/toycar/urdf_description/robot_core0.xacro (robot description, xacro)
@@ -41,4 +41,7 @@
         </xacro:inertial_box>
     </link>
+    <gazebo reference = "chassis">
+    <material>Gazebo/White</material>
+    </gazebo>
     <!-- LEFT WHEEL LINK -->
     <joint name="left_wheel_joint" type="continuous">
@@ -64,4 +67,7 @@
         </xacro:inertial_cylinder>
     </link>
+    <gazebo reference = "left_wheel">
+    <material>Gazebo/Grey</material>
+    </gazebo>
     <!-- RIGHT WHEEL LINK -->
     <joint name="right_wheel_joint" type="continuous">
@@ -87,4 +93,7 @@
         </xacro:inertial_cylinder>
     </link>
+    <gazebo reference = "right_wheel">
+    <material>Gazebo/Grey</material>
+    </gazebo>
     <!-- CASTER WHEEL LINK -->
     <joint name="caster_wheel_joint" type="fixed">
@@ -109,3 +118,6 @@
         </xacro:inertial_sphere>
     </link>
+    <gazebo reference = "caster_wheel">
+    <material>Gazebo/Grey</material>
+    </gazebo>
 </robot>

File: ros_ws/scr/toycar/urdf_description/robot_core.xacro (robot description, xacro)
@@ -42,5 +42,5 @@
     </link>
     <gazebo reference = "chassis">
-    <material>Gazebo/white    </material>
+    <material>Gazebo/White</material>
     </gazebo>
     <!-- LEFT WHEEL LINK -->
@@ -68,5 +68,5 @@
     </link>
     <gazebo reference = "left_wheel">
-    <material>Gazebo/grey</material>
+    <material>Gazebo/Grey</material>
     </gazebo>
     <!-- RIGHT WHEEL LINK -->
@@ -119,5 +119,5 @@
     </link>
     <gazebo reference = "left_wheel">
-    <material>Gazebo/grey</material>
+    <material>Gazebo/Grey</material>
     </gazebo>
 </robot>
