Commit message: Failed GPU sensor

File: ros_ws/install/toycar/share/toycar/urdf_description/diff_drive.xacro (robot description, xacro)
@@ -1,21 +1,24 @@
 <?xml version="1.0"?>
 <robot xmlns:xacro="http://www.ros.org/wiki/xacro" >
-<gazebo>
-    <plugin name= "diff_drive" filename = "libgazebo_ros_diff_drive.so">
-            <!-- wheel info -->
-        <left_joint>left_wheel_joint</left_joint>
-        <right_joint>right_wheel_joint</right_joint>
-        <wheel_separation>0.35</wheel_separation>
-        <wheel_diameter>0.35</wheel_diameter>
-            <!-- limits -->
-        <max_wheel_toque>100</max_wheel_toque>
-        <max_wheel_acceleration>3.9</max_wheel_acceleration>
-            <!-- Output -->
-        <odometry_frame>odom</odometry_frame>
-        <robot_base_frame>baselink</robot_base_frame>
-        <publish_odom>true</publish_odom>
-        <publish_odom_tf>true</publish_odom_tf>
-        <publish_wheel_tf>true</publish_wheel_tf>
-    </plugin>
-</gazebo>
+    <gazebo>
+        <plugin name= "diff_drive_controller" filename = "libgazebo_ros_diff_drive.so">
+            <!-- general settings -->
+            <alwaysOn>true</alwaysOn>
+            <updateRate>20</updateRate>
+                <!-- wheel info -->
+            <left_joint>left_wheel_joint</left_joint>
+            <right_joint>right_wheel_joint</right_joint>
+            <wheel_separation>0.35</wheel_separation>
+            <wheel_diameter>0.35</wheel_diameter>
+                <!-- limits -->
+            <max_wheel_toque>100</max_wheel_toque>
+            <max_wheel_acceleration>3.9</max_wheel_acceleration>
+                <!-- Output -->
+            <odometry_frame>odom</odometry_frame>
+            <robot_base_frame>baselink</robot_base_frame>
+            <publish_odom>true</publish_odom>
+            <publish_odom_tf>true</publish_odom_tf>
+            <publish_wheel_tf>true</publish_wheel_tf>
+        </plugin>
+    </gazebo>
 </robot>

File: ros_ws/install/toycar/share/toycar/urdf_description/robot.urdf.xacro (robot description, xacro)
@@ -3,3 +3,4 @@
 <xacro:include filename="robot_core0.xacro" />
 <xacro:include filename="diff_drive.xacro" />
+<xacro:include filename="lidar.xacro" />
 </robot>

File: ros_ws/install/toycar/share/toycar/urdf_description/robot_core.xacro (robot description, xacro)
@@ -13,4 +13,8 @@
     <material name="black">
         <color rgba="0 0 0 1"/>
+    </material>
+    <material name ="red">
+        <color rgba = "1 0 0 1">
+        </color>
     </material>
     <!-- BASE LINK -->
@@ -43,4 +47,7 @@
     <gazebo reference = "chassis">
     <material>Gazebo/White</material>
+    </gazebo>
+    <gazebo reference = "lidar_link">
+    <material>Gazebo/Green</material>
     </gazebo>
     <!-- LEFT WHEEL LINK -->
@@ -118,6 +125,8 @@
         </xacro:inertial_sphere>
     </link>
-    <gazebo reference = "left_wheel">
+    <gazebo reference = "caster_wheel">
     <material>Gazebo/Grey</material>
+    <mu1 value="0.0001" />
+    <mu2 value="0.0001" />
     </gazebo>
 </robot>

File: ros_ws/install/toycar/share/toycar/urdf_description/robot_core0.xacro (robot description, xacro)
@@ -13,4 +13,8 @@
     <material name="black">
         <color rgba="0 0 0 1"/>
+    </material>
+    <material name ="red">
+        <color rgba = "1 0 0 1">
+        </color>
     </material>
     <!-- BASE LINK -->
@@ -43,4 +47,7 @@
     <gazebo reference = "chassis">
     <material>Gazebo/White</material>
+    </gazebo>
+    <gazebo reference = "lidar_link">
+    <material>Gazebo/Green</material>
     </gazebo>
     <!-- LEFT WHEEL LINK -->
@@ -120,4 +127,6 @@
     <gazebo reference = "caster_wheel">
     <material>Gazebo/Grey</material>
+    <mu1 value="0.0001" />
+    <mu2 value="0.0001" />
     </gazebo>
 </robot>
