Commit message: laser scaner pluig has refuse completely to work

File: ros_ws/install/toycar/share/toycar/urdf_description/lidar.xacro (robot description, xacro)
@@ -24,5 +24,5 @@
         </xacro:inertial_cylinder>
     </link>
-    <gazebo reference = "lidar_joint">
+    <!-- <gazebo reference = "lidar_joint">
     <material>Gazebo/Red</material>
             <sensor type="ray" name="laser">
@@ -44,15 +44,11 @@
                         <resolution>0.01</resolution>
                     </range>
-                    <!-- <noise>
+                    <noise>
                     <type>gaussian</type>
-                    Noise parameters based on published spec for Hokuyo laser
-                        achieving "+-30mm" accuracy at range < 10m.  A mean of 0.0m and
-                        stddev of 0.01m will put 99.7% of samples within 0.03m of the true
-                        reading.
                     <mean>0.0</mean>
                     <stddev>0.01</stddev>
-                    </noise> -->
+                    </noise>
                 </ray>
-                <plugin name="laser_controller" filename="libgazebo_ros_laser.so">
+                <plugin name="laser_controller" filename="libgazebo_ros_ray_sensor.so">
                     <ros>
                         <argument>
@@ -61,8 +57,80 @@
                     </ros>
                     <output_type>sensor_msgs/Laserscan</output_type>
-                    <topic_name>/rrbot/laser/scan</topic_name>
-                    <frame_name>laser_frame</frame_name>
+                     <frame_name>laser_frame</frame_name>
                 </plugin>
             </sensor>
     </gazebo>
+     -->
+     <!-- <gazebo>
+  <plugin name="camera_plugin" filename="libgazebo_ros_camera.so">
+    <alwaysOn>true</alwaysOn>
+    <updateRate>30.0</updateRate>
+    <cameraName>camera</cameraName>
+    <imageTopicName>image_raw</imageTopicName>
+    <cameraInfoTopicName>camera_info</cameraInfoTopicName>
+    <hackBaseline>0.07</hackBaseline>
+    <distortionK1>0.0</distortionK1>
+    <distortionK2>0.0</distortionK2>
+    <distortionK3>0.0</distortionK3>
+    <distortionT1>0.0</distortionT1>
+    <distortionT2>0.0</distortionT2>
+  </plugin>
+  <sensor name="camera" type="camera">
+    <camera name="camera">
+      <horizontal_fov>1.047</horizontal_fov>
+      <image>
+        <width>640</width>
+        <height>480</height>
+        <format>R8G8B8</format>
+      </image>
+      <clip>
+        <near>0.1</near>
+        <far>1000</far>
+      </clip>
+      <noise>
+        <type>gaussian</type>
+        <mean>0.0</mean>
+        <stddev>0.01</stddev>
+      </noise>
+      <distortion>k1 k2 p1 p2 k3 0 0 0 0 0</distortion>
+      <pose frame=''>0 0 1.5 0 -1.57 3.14</pose>
+    </camera>
+    <always_on>true</always_on>
+    <update_rate>30.0</update_rate>
+    <visualize>true</visualize>
+  </sensor>
+</gazebo> -->
+<gazebo reference="lidar_joint">
+  <sensor type="gpu_ray" name="head_hokuyo_sensor">
+    <pose>0 0 0.09 1.5708 0 -1.5708</pose>
+    <visualize>true</visualize>
+    <update_rate>30</update_rate>
+    <ray>
+     <noise>
+      <type>gaussian</type>
+      <mean>0.0</mean>
+      <stddev>0.1</stddev>
+     </noise>
+      <scan>
+        <horizontal>
+          <samples>32</samples>
+          <resolution>1</resolution>
+          <min_angle>-0.53529248</min_angle>
+          <max_angle>0.18622663
+</max_angle>
+        </horizontal>
+      </scan>
+      <range>
+        <min>0.05</min>
+        <max>70</max>
+        <resolution>0.02</resolution>
+      </range>
+    </ray>
+    <plugin name="hokuyo_node" filename="libgazebo_ros_ray_sensor.so">
+     <!-- or libgazebo_ros_gpu_laser -->
+      <topicName>/myrobot1/laser/scan</topicName>
+      <frameName>base</frameName>
+    </plugin>
+  </sensor>
+</gazebo>
 </robot>

File: ros_ws/scr/toycar/urdf_description/lidar.xacro (robot description, xacro)
@@ -44,15 +44,11 @@
                         <resolution>0.01</resolution>
                     </range>
-                    <!-- <noise>
+                    <noise>
                     <type>gaussian</type>
-                    Noise parameters based on published spec for Hokuyo laser
-                        achieving "+-30mm" accuracy at range < 10m.  A mean of 0.0m and
-                        stddev of 0.01m will put 99.7% of samples within 0.03m of the true
-                        reading.
                     <mean>0.0</mean>
                     <stddev>0.01</stddev>
-                    </noise> -->
+                    </noise>
                 </ray>
-                <plugin name="laser_controller" filename="libgazebo_ros_laser.so">
+                <plugin name="laser_controller" filename="libgazebo_ros_ray_sensor.so">
                     <ros>
                         <argument>

File: ros_ws/scr/toycar/urdf_description/robot_core0.xacro (robot description, xacro)
@@ -19,6 +19,5 @@
     </material>
     <!-- BASE LINK -->
-    <link name="base_link">
-    </link>
+    <link name="base_link" />
     <!-- CHASSIS LINK -->
     <joint name="chassis_joint" type="fixed">

Commit message: laser worked working on using turbot3 house world

File: ros_ws/install/toycar/share/toycar/urdf_description/lidar.xacro (robot description, xacro)
@@ -24,5 +24,5 @@
         </xacro:inertial_cylinder>
     </link>
-    <!-- <gazebo reference = "lidar_joint">
+    <gazebo reference = "lidar_link">
     <material>Gazebo/Red</material>
             <sensor type="ray" name="laser">
@@ -60,77 +60,38 @@
                 </plugin>
             </sensor>
+            <!-- <sensor name="hls_lfcd_lds" type="ray">
+        <always_on>true</always_on>
+        <visualize>true</visualize>
+        <pose>-0.064 0 0.121 0 0 0</pose>
+        <update_rate>5</update_rate>
+        <ray>
+          <scan>
+            <horizontal>
+              <samples>360</samples>
+              <resolution>1.000000</resolution>
+              <min_angle>0.000000</min_angle>
+              <max_angle>6.280000</max_angle>
+            </horizontal>
+          </scan>
+          <range>
+            <min>0.120000</min>
+            <max>3.5</max>
+            <resolution>0.015000</resolution>
+          </range>
+          <noise>
+            <type>gaussian</type>
+            <mean>0.0</mean>
+            <stddev>0.01</stddev>
+          </noise>
+        </ray>
+        <plugin name="turtlebot3_laserscan" filename="libgazebo_ros_ray_sensor.so">
+          <ros>
+ #########           <namespace>/tb3</namespace>
+            <remapping>~/out:=scan</remapping>
+          </ros>
+          <output_type>sensor_msgs/LaserScan</output_type>
+          <frame_name>base_scan</frame_name>
+        </plugin>
+      </sensor> -->
     </gazebo>
-     -->
-     <!-- <gazebo>
-  <plugin name="camera_plugin" filename="libgazebo_ros_camera.so">
-    <alwaysOn>true</alwaysOn>
-    <updateRate>30.0</updateRate>
-    <cameraName>camera</cameraName>
-    <imageTopicName>image_raw</imageTopicName>
-    <cameraInfoTopicName>camera_info</cameraInfoTopicName>
-    <hackBaseline>0.07</hackBaseline>
-    <distortionK1>0.0</distortionK1>
-    <distortionK2>0.0</distortionK2>
-    <distortionK3>0.0</distortionK3>
-    <distortionT1>0.0</distortionT1>
-    <distortionT2>0.0</distortionT2>
-  </plugin>
-  <sensor name="camera" type="camera">
-    <camera name="camera">
-      <horizontal_fov>1.047</horizontal_fov>
-      <image>
-        <width>640</width>
-        <height>480</height>
-        <format>R8G8B8</format>
-      </image>
-      <clip>
-        <near>0.1</near>
-        <far>1000</far>
-      </clip>
-      <noise>
-        <type>gaussian</type>
-        <mean>0.0</mean>
-        <stddev>0.01</stddev>
-      </noise>
-      <distortion>k1 k2 p1 p2 k3 0 0 0 0 0</distortion>
-      <pose frame=''>0 0 1.5 0 -1.57 3.14</pose>
-    </camera>
-    <always_on>true</always_on>
-    <update_rate>30.0</update_rate>
-    <visualize>true</visualize>
-  </sensor>
-</gazebo> -->
-<gazebo reference="lidar_joint">
-  <sensor type="gpu_ray" name="head_hokuyo_sensor">
-    <pose>0 0 0.09 1.5708 0 -1.5708</pose>
-    <visualize>true</visualize>
-    <update_rate>30</update_rate>
-    <ray>
-     <noise>
-      <type>gaussian</type>
-      <mean>0.0</mean>
-      <stddev>0.1</stddev>
-     </noise>
-      <scan>
-        <horizontal>
-          <samples>32</samples>
-          <resolution>1</resolution>
-          <min_angle>-0.53529248</min_angle>
-          <max_angle>0.18622663
-</max_angle>
-        </horizontal>
-      </scan>
-      <range>
-        <min>0.05</min>
-        <max>70</max>
-        <resolution>0.02</resolution>
-      </range>
-    </ray>
-    <plugin name="hokuyo_node" filename="libgazebo_ros_ray_sensor.so">
-     <!-- or libgazebo_ros_gpu_laser -->
-      <topicName>/myrobot1/laser/scan</topicName>
-      <frameName>base</frameName>
-    </plugin>
-  </sensor>
-</gazebo>
 </robot>

File: ros_ws/install/toycar/share/toycar/urdf_description/robot_core0.xacro (robot description, xacro)
@@ -19,6 +19,12 @@
     </material>
     <!-- BASE LINK -->
-    <link name="base_link">
-    </link>
+    <link name="base_link" />
+    <!-- Base foot print -->
+    <joint  name="base_footprint" type="fixed">
+    <parent link="base_link" />
+    <child link="base_footprint" />
+    <origin xyz = "0 0 0" rpy = "0 0 0" />
+    </joint>
+    <link name="base_footprint"/>
     <!-- CHASSIS LINK -->
     <joint name="chassis_joint" type="fixed">
@@ -48,7 +54,7 @@
     <material>Gazebo/White</material>
     </gazebo>
-    <gazebo reference = "lidar_link">
+    <!-- <gazebo reference = "lidar_link">
     <material>Gazebo/Green</material>
-    </gazebo>
+    </gazebo> -->
     <!-- LEFT WHEEL LINK -->
     <joint name="left_wheel_joint" type="continuous">

File: ros_ws/scr/toycar/urdf_description/lidar.xacro (robot description, xacro)
@@ -24,5 +24,5 @@
         </xacro:inertial_cylinder>
     </link>
-    <gazebo reference = "lidar_joint">
+    <gazebo reference = "lidar_link">
     <material>Gazebo/Red</material>
             <sensor type="ray" name="laser">
@@ -60,4 +60,38 @@
                 </plugin>
             </sensor>
+            <!-- <sensor name="hls_lfcd_lds" type="ray">
+        <always_on>true</always_on>
+        <visualize>true</visualize>
+        <pose>-0.064 0 0.121 0 0 0</pose>
+        <update_rate>5</update_rate>
+        <ray>
+          <scan>
+            <horizontal>
+              <samples>360</samples>
+              <resolution>1.000000</resolution>
+              <min_angle>0.000000</min_angle>
+              <max_angle>6.280000</max_angle>
+            </horizontal>
+          </scan>
+          <range>
+            <min>0.120000</min>
+            <max>3.5</max>
+            <resolution>0.015000</resolution>
+          </range>
+          <noise>
+            <type>gaussian</type>
+            <mean>0.0</mean>
+            <stddev>0.01</stddev>
+          </noise>
+        </ray>
+        <plugin name="turtlebot3_laserscan" filename="libgazebo_ros_ray_sensor.so">
+          <ros>
+ #########           <namespace>/tb3</namespace>
+            <remapping>~/out:=scan</remapping>
+          </ros>
+          <output_type>sensor_msgs/LaserScan</output_type>
+          <frame_name>base_scan</frame_name>
+        </plugin>
+      </sensor> -->
     </gazebo>
 </robot>

File: ros_ws/scr/toycar/urdf_description/robot_core0.xacro (robot description, xacro)
@@ -20,4 +20,11 @@
     <!-- BASE LINK -->
     <link name="base_link" />
+    <!-- Base foot print -->
+    <joint  name="base_footprint" type="fixed">
+    <parent link="base_link" />
+    <child link="base_footprint" />
+    <origin xyz = "0 0 0" rpy = "0 0 0" />
+    </joint>
+    <link name="base_footprint"/>
     <!-- CHASSIS LINK -->
     <joint name="chassis_joint" type="fixed">
@@ -47,7 +54,7 @@
     <material>Gazebo/White</material>
     </gazebo>
-    <gazebo reference = "lidar_link">
+    <!-- <gazebo reference = "lidar_link">
     <material>Gazebo/Green</material>
-    </gazebo>
+    </gazebo> -->
     <!-- LEFT WHEEL LINK -->
     <joint name="left_wheel_joint" type="continuous">

Commit message: Abstacle avoidence implemented

File: ros_ws/install/toycar/share/toycar/urdf_description/lidar.xacro (robot description, xacro)
@@ -4,5 +4,5 @@
         <parent link="base_link"/>
         <child link="lidar_link"/>
-        <origin xyz="0.17 0 0.15"/>
+        <origin xyz="0.05 0 0.15"/>
     </joint>
     <link name="lidar_link">
@@ -33,12 +33,12 @@
                     <scan>
                     <horizontal>
-                        <samples>400</samples>
+                        <samples>500</samples>
                         <resolution>1</resolution>
-                        <min_angle>-3.14</min_angle>
-                        <max_angle>3.14</max_angle>
+                        <min_angle>-1.578796</min_angle>
+                        <max_angle>1.578796</max_angle>
                     </horizontal>
                     </scan>
                     <range>
-                        <min>0.320</min>
+                        <min>.2245</min>
                         <max>12.0</max>
                         <resolution>0.02</resolution>
